Commit message: Fixed.

File: src/gae_launch/urdf/sensors.urdf.xacro (robot description, xacro)
@@ -9,6 +9,6 @@
     <parent link="base_link"/>
     <child link="gnss_link2"/>
-    <!-- x=+1m (ön), y=+0.65m (sol), z=1.0m yükseklik -->
-    <origin xyz="2.0 0.65 1.0" rpy="0 0 0"/>
+    <!-- x=+1m (ön), y=-0.65m (sol), z=1.0m yükseklik -->
+    <origin xyz="1.0 -0.65 1.0" rpy="0 0 0"/>
   </joint>
   <!-- Rear-Left GNSS -->
@@ -18,7 +18,6 @@
     <child link="gnss_link"/>
     <!-- x=–1m (arka), y=+0.65m (sol), z=1.0m yükseklik -->
-    <origin xyz="0.0 0.65 1.0" rpy="0 0 0"/>
+    <origin xyz="-1.0 -0.65 1.0" rpy="0 0 0"/>
   </joint>
-  <!-- IMU Sensörleri -->
   <!-- Front-Right IMU -->
   <link name="imu_link2"/>
